File: Smart Fragrance.kicad_sch (KiCad schematic)
At the start: 18 parts, among them J1 STM_PROGRAMER_PRT-14417, U1 LIS3DHTR, U2 STM32L031G6U6TR, U4 B3FS-1010

Commit message: layout is done
Parts:
- renumbered U4 to U3
Connections:
- net GND: no longer R2.1, R2.2
- net LED: now also R2.1, R2.2
Other:
- moved on the sheet: R2
Changed lines of the file:
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@@
 	)
 	(junction
+		(at 91.44 113.03)
+		(diameter 0)
+		(color 0 0 0 0)
+	)
+	(junction
 		(at 228.6 87.63)
 		(diameter 0)
@@
 	(wire
 		(pts
-			(xy 95.25 121.92) (xy 86.36 121.92)
+			(xy 86.36 121.92) (xy 106.68 121.92)
 		)
 		(stroke
@@
 	(wire
 		(pts
+			(xy 91.44 113.03) (xy 81.28 113.03)
+		)
+		(stroke
+			(width 0.6604)
+			(type default)
+		)
+	)
+	(wire
+		(pts
 			(xy 156.21 100.33) (xy 152.4 100.33)
 		)
@@
 	(wire
 		(pts
-			(xy 120.65 113.03) (xy 81.28 113.03)
+			(xy 120.65 113.03) (xy 105.41 113.03)
 		)
 		(stroke
@@
 	(wire
 		(pts
+			(xy 91.44 113.03) (xy 91.44 116.84)
+		)
+		(stroke
+			(width 0)
+			(type default)
+		)
+	)
+	(wire
+		(pts
 			(xy 43.18 63.5) (xy 57.15 63.5)
 		)
@@
 	(wire
 		(pts
+			(xy 97.79 113.03) (xy 91.44 113.03)
+		)
+		(stroke
+			(width 0.6604)
+			(type default)
+		)
+	)
+	(wire
+		(pts
 			(xy 48.26 45.72) (xy 44.45 45.72)
 		)
@@
 	(wire
 		(pts
-			(xy 106.68 121.92) (xy 102.87 121.92)
-		)
-		(stroke
-			(width 0.6604)
-			(type default)
-		)
-	)
-	(wire
-		(pts
 			(xy 113.03 121.92) (xy 106.68 121.92)
 		)
@@
 		)
 	)
+	(label "LED"
+		(at 91.44 116.84 0)
+		(fields_autoplaced yes)
+		(effects
+			(font
+				(size 1.524 1.524)
+			)
+			(justify left bottom)
+		)
+		(property "Netclass" "LED"
+			(at 91.44 118.745 0)
+			(effects
+				(font
+					(size 1.524 1.524)
+					(italic yes)
+				)
+				(justify left)
+			)
+		)
+	)
 	(label "NSS_CS"
 		(at 57.15 40.64 0)
@@
 		(on_board yes)
 		(dnp no)
-		(property "Reference" "#PWR015"
+		(property "Reference" "#PWR013"
 			(at 180.34 109.22 0)
 			(effects
@@
 			(project "Smart Fragrance"
 				(path "/9741c116-8e46-4487-9d70-0fa4b07a3868"
-					(reference "#PWR015")
+					(reference "#PWR013")
 					(unit 1)
 				)
@@
 		(on_board yes)
 		(dnp no)
-		(property "Reference" "#PWR05"
+		(property "Reference" "#PWR04"
 			(at 63.5 101.6 0)
 			(effects
@@
 			(project "Smart Fragrance"
 				(path "/9741c116-8e46-4487-9d70-0fa4b07a3868"
-					(reference "#PWR05")
+					(reference "#PWR04")
 					(unit 1)
 				)
@@
 		(dnp no)
 		(fields_autoplaced yes)
-		(property "Reference" "#PWR08"
+		(property "Reference" "#PWR07"
 			(at 143.51 133.35 0)
 			(effects
@@
 			(project "Smart Fragrance"
 				(path "/9741c116-8e46-4487-9d70-0fa4b07a3868"
-					(reference "#PWR08")
+					(reference "#PWR07")
 					(unit 1)
 				)
@@
 		(dnp no)
 		(fields_autoplaced yes)
-		(property "Reference" "#PWR09"
+		(property "Reference" "#PWR08"
 			(at 147.32 151.13 0)
 			(effects
@@
 			(project "Smart Fragrance"
 				(path "/9741c116-8e46-4487-9d70-0fa4b07a3868"
-					(reference "#PWR09")
+					(reference "#PWR08")
 					(unit 1)
 				)
@@
 		(on_board yes)
 		(dnp no)
-		(property "Reference" "#PWR010"
+		(property "Reference" "#PWR09"
 			(at 156.21 151.13 0)
 			(effects
@@
 			(project "Smart Fragrance"
 				(path "/9741c116-8e46-4487-9d70-0fa4b07a3868"
-					(reference "#PWR010")
+					(reference "#PWR09")
 					(unit 1)
 				)
@@
 		(dnp no)
 		(fields_autoplaced yes)
-		(property "Reference" "#PWR06"
+		(property "Reference" "#PWR05"
 			(at 116.84 149.86 0)
 			(effects
@@
 			(project "Smart Fragrance"
 				(path "/9741c116-8e46-4487-9d70-0fa4b07a3868"
-					(reference "#PWR06")
+					(reference "#PWR05")
 					(unit 1)
 				)
@@
 		(on_board yes)
 		(dnp no)
-		(property "Reference" "#PWR04"
+		(property "Reference" "#PWR03"
 			(at 48.26 57.15 0)
 			(effects
@@
 			(project "Smart Fragrance"
 				(path "/9741c116-8e46-4487-9d70-0fa4b07a3868"
-					(reference "#PWR04")
+					(reference "#PWR03")
 					(unit 1)
 				)
@@
 		(dnp no)
 		(fields_autoplaced yes)
-		(property "Reference" "#PWR012"
+		(property "Reference" "#PWR011"
 			(at 163.83 151.13 0)
 			(effects
@@
 			(project "Smart Fragrance"
 				(path "/9741c116-8e46-4487-9d70-0fa4b07a3868"
-					(reference "#PWR012")
+					(reference "#PWR011")
 					(unit 1)
 				)
@@
 	(symbol
 		(lib_id "Device:R_US")
-		(at 99.06 121.92 90)
+		(at 101.6 113.03 90)
 		(unit 1)
 		(exclude_from_sim no)
@@
 		(fields_autoplaced yes)
 		(property "Reference" "R2"
-			(at 99.06 115.57 90)
+			(at 101.6 106.68 90)
 			(effects
 				(font
@@
 		)
 		(property "Value" "330"
-			(at 99.06 118.11 90)
+			(at 101.6 109.22 90)
 			(effects
 				(font
@@
 		)
 		(property "Footprint" "Resistor_SMD:R_0402_1005Metric"
-			(at 99.314 120.904 90)
+			(at 101.854 112.014 90)
 			(effects
 				(font
@@
 		)
 		(property "Datasheet" "https://www.yageo.com/upload/media/product/products/datasheet/rchip/PYu-RC_Group_51_RoHS_L_12.pdf"
-			(at 99.06 121.92 0)
+			(at 101.6 113.03 0)
 			(effects
 				(font
@@
 		)
 		(property "Description" "RES 330 OHM 5% 1/10W 0603"
-			(at 99.06 121.92 0)
+			(at 101.6 113.03 0)
 			(effects
 				(font
@@
 		)
 		(property "Digikey" "311-330GRCT-ND"
-			(at 99.06 121.92 90)
+			(at 101.6 113.03 90)
 			(effects
 				(font
@@
 		)
 		(property "Manufacturer" "YAGEO"
-			(at 99.06 121.92 90)
+			(at 101.6 113.03 90)
 			(effects
 				(font
@@
 		)
 		(property "Mfg part #" "RC0603JR-07330RL"
-			(at 99.06 121.92 90)
+			(at 101.6 113.03 90)
 			(effects
 				(font
@@
 		)
 		(instances
-			(project ""
+			(project "Smart Fragrance"
 				(path "/9741c116-8e46-4487-9d70-0fa4b07a3868"
 					(reference "R2")
@@
 		(dnp no)
 		(fields_autoplaced yes)
-		(property "Reference" "U4"
+		(property "Reference" "U3"
 			(at 207.01 77.47 0)
 			(effects
@@
 			(project ""
 				(path "/9741c116-8e46-4487-9d70-0fa4b07a3868"
-					(reference "U4")
+					(reference "U3")
 					(unit 1)
 				)
@@
 		(dnp no)
 		(fields_autoplaced yes)
-		(property "Reference" "#PWR013"
+		(property "Reference" "#PWR012"
 			(at 172.72 151.13 0)
 			(effects
@@
 			(project "Smart Fragrance"
 				(path "/9741c116-8e46-4487-9d70-0fa4b07a3868"
-					(reference "#PWR013")
+					(reference "#PWR012")
 					(unit 1)
 				)
@@
 		(on_board yes)
 		(dnp no)
-		(property "Reference" "#PWR07"
+		(property "Reference" "#PWR06"
 			(at 134.62 133.35 0)
 			(effects
@@
 			(project "Smart Fragrance"
 				(path "/9741c116-8e46-4487-9d70-0fa4b07a3868"
-					(reference "#PWR07")
+					(reference "#PWR06")
 					(unit 1)
 				)
@@
 		(dnp no)
 		(fields_autoplaced yes)
-		(property "Reference" "#PWR011"
+		(property "Reference" "#PWR010"
 			(at 160.02 90.17 0)
 			(effects
@@
 			(project ""
 				(path "/9741c116-8e46-4487-9d70-0fa4b07a3868"
-					(reference "#PWR011")
+					(reference "#PWR010")
 					(unit 1)
 				)
@@
 		(dnp no)
 		(fields_autoplaced yes)
-		(property "Reference" "#PWR016"
+		(property "Reference" "#PWR014"
 			(at 233.68 93.98 0)
 			(effects
@@
 			(project "Smart Fragrance"
 				(path "/9741c116-8e46-4487-9d70-0fa4b07a3868"
-					(reference "#PWR016")
+					(reference "#PWR014")
 					(unit 1)
 				)
